File: Hydro 4/High voltage clamper/High voltage clamper.kicad_pcb (KiCad board)
At the start: 0 parts

Commit message: added PCB
Parts:
- added D1: ZMDxx, Diode_SMD:D_MiniMELF, F.Cu at (124.3, 96.1)
- added Q1: IRF740, Package_TO_SOT_THT:TO-220-3_Vertical, F.Cu at (146.1, 88.5)
Routing:
- net -VDC: track 0.00 -> 28.2 mm
- net Net-(D1-K): track 0.00 -> 26.6 mm
Other:
- copper layers 0 -> 2
